File: power supply v3/pwrv3.kicad_pcb (KiCad board)
At the start: 2 copper layers, 38.3 x 37.5 mm, 56 parts, among them IC1 TLV3701IDBVR, IC2 LM25145RGYR, IC3 LMR50410YQDBVRQ1, J1 1.5 mm, J3 1933189, J4 Conn_01x04_Pin 1.27mm, Q1 35A, 30V, Q2 35A Id, 30V Vds

Commit message: tous les noms
Other:
- board text added: "Ambre"
- board text added: "Julien"
Changed lines of the file:
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@@
+		)
+	)
+	(gr_text "Julien"
+		(at 197.04 110.54 0)
+		(layer "B.SilkS")
+		(effects
+			(font
+				(size 0.8 0.8)
+				(thickness 0.16)
+				(bold yes)
+			)
+			(justify left bottom mirror)
+		)
+	)
+	(gr_text "Ambre"
+		(at 192.89 110.54 0)
+		(layer "B.SilkS")
+		(effects
+			(font
+				(size 0.8 0.8)
+				(thickness 0.16)
+				(bold yes)
+			)
+			(justify left bottom mirror)
 		)
 	)
